Commit message: Fixed minor spelling mistake (jont -> joint)

File: hooks/samples/xml/valid/bender.urdf (robot description, URDF)
Before this commit: robot bender, 49 links, 48 joints
Joints:
- removed joint base_fixed_jont
- removed joint body_fixed_jont
- added joint base_fixed_joint: type fixed, parent bender/base_link, child bender/base_footprint, origin xyz=0 0 0 rpy=0 0 0, axis 0 0 0
- added joint body_fixed_joint: type fixed, parent bender/base_link, child bender/body, origin xyz=0 0 0 rpy=0 0 0, axis 0 0 0
